File: boards/TARS-MK4/TARS-MK4-PMB-TEMPLATE1/BATTERY.kicad_sch (KiCad schematic)
At the start: 0 parts

Commit message: continued making template
Other:
- note added: "stuff relating to all stuff battery, including charging."
Changed lines of the file:
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@@
 (kicad_sch (version 20211123) (generator eeschema)
   (paper "A4")
+  (text "stuff relating to all stuff battery, including charging."
+    (at 111.125 83.185 0)
+    (effects (font (size 1.27 1.27) italic) (justify left bottom))
+  )
 )
