File: boards/TARS-MK4/TARS-MK4-PMB-TEMPLATE1/MCU.kicad_sch (KiCad schematic)
At the start: 0 parts

Commit message: continued making template
Other:
- note added: "CONTROLLER"
- note added: "FLASH"
Changed lines of the file:
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@@
 (kicad_sch (version 20211123) (generator eeschema)
   (paper "A4")
-  (polyline (pts (xy 20.955 19.685) (xy 20.955 61.595))
+  (polyline (pts (xy 79.375 24.765) (xy 79.375 87.63))
     (stroke (width 0) (type default) (color 0 0 0 0))
   )
-  (polyline (pts (xy 20.955 61.595) (xy 64.135 61.595))
+  (polyline (pts (xy 176.53 123.19) (xy 88.9 123.19))
     (stroke (width 0) (type default) (color 0 0 0 0))
   )
-  (polyline (pts (xy 64.135 61.595) (xy 64.135 19.685))
+  (polyline (pts (xy 88.9 24.765) (xy 176.53 24.765))
     (stroke (width 0) (type default) (color 0 0 0 0))
   )
-  (polyline (pts (xy 20.955 19.685) (xy 64.135 19.685))
+  (polyline (pts (xy 17.78 24.765) (xy 79.375 24.765))
     (stroke (width 0) (type default) (color 0 0 0 0))
   )
+  (polyline (pts (xy 79.375 87.63) (xy 17.78 87.63))
+    (stroke (width 0) (type default) (color 0 0 0 0))
+  )
+  (polyline (pts (xy 176.53 24.765) (xy 176.53 123.19))
+    (stroke (width 0) (type default) (color 0 0 0 0))
+  )
+  (polyline (pts (xy 17.78 24.765) (xy 17.78 87.63))
+    (stroke (width 0) (type default) (color 0 0 0 0))
+  )
+  (polyline (pts (xy 88.9 24.765) (xy 88.9 123.19))
+    (stroke (width 0) (type default) (color 0 0 0 0))
+  )
+  (text "FLASH" (at 17.78 24.765 0)
+    (effects (font (size 5 5) italic) (justify left bottom))
+  )
+  (text "CONTROLLER" (at 88.9 24.765 0)
+    (effects (font (size 5 5) italic) (justify left bottom))
+  )
 )
