File: boards/TARS-MK3/TARS-MK3-FCB_v3.1/FCB.kicad_sch (KiCad schematic)
At the start: 4 parts, among them J1 Conn_02x12_Odd_Even, J2 Conn_02x12_Odd_Even, J3 Conn_02x12_Odd_Even, J4 Conn_02x12_Odd_Even

Commit message: added names to FCB sheets
Other:
- title: (none) -> TARS Flight Computer Schematic
Changed lines of the file:
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@@
 (kicad_sch (version 20211123) (generator eeschema)
   (paper "A4")
+  (title_block
+    (title "TARS Flight Computer Schematic")
+    (date "2022-09-06")
+    (rev "3.1")
+  )
   (polyline (pts (xy 105.41 16.51) (xy 105.41 161.29))
     (stroke (width 0) (type default) (color 0 0 0 0))
