File: boards/TARS-MK3/TARS-MK3-TELEM_v3.1/TELEM.kicad_pcb (KiCad board)
At the start: 2 copper layers, 86 x 79.1 mm, 15 parts, among them J101 Conn_02x12_Odd_Even, J102 Conn_02x12_Odd_Even, J103 Conn_02x12_Odd_Even, J104 Conn_02x12_Odd_Even, J105 2091680401, J106 536270474

Commit message: aligned B2bs
Parts:
- removed the J101 at (30.0, -7.00)
- removed the J102 at (30.0, -7.00)
- removed the J103 at (-30.0, -7.00)
- removed the J104 at (-30.0, -7.00)
- J102, J104: moved to B.Cu
- J105: value 2091680401 -> Receptacle
- moved J103 167.0 mm to (-30.0, -7.00)
- moved J104 155.4 mm to (-30.0, -7.00), turned to 180 degrees
- moved J101 125.6 mm to (30.0, -7.00), turned to 180 degrees
- moved J102 95.9 mm to (30.0, -7.00)
