File: boards/TARS-MK3/TARS-MK3-PMB_v3.1/3V3_REG.kicad_sch (KiCad schematic)
At the start: 0 parts

Commit message: Updated Symbol of 3V3 Regulator. Designed schematic for 3V3 regulator
Parts:
- added Cin: 1 uF, symbol Device:C
- added Cout: 22uF, symbol Device:C
- added Cvcc: 1uF, symbol Device:C
- added L1: 68uH, symbol pspice:INDUCTOR
- added U?: MAX17640AATA, symbol Regulator_Switching_MAX17640AATA:MAX17640AATA
Connections:
- new net: Cvcc.1, U?.3 (Vcc)
- new net: L1.1, U?.8 (LX)
- new net 3V3_REG_RESET: U?.6 (RESET)
- new net GND: Cin.2, Cout.2, Cvcc.2, U?.7 (GND)
- new net Mode 3V3: U?.5 (MODE)
- new net V bat: Cin.1, U?.1 (Vin), U?.2 (EN/UVLO)
- new net Vout 3.3V: Cout.1, L1.2, U?.4 (Vout)
Changed lines of the file:
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@@
     (rev "3.1")
   )
+  (junction (at 88.9 52.07) (diameter 0) (color 0 0 0 0)
+  )
+  (junction (at 139.7 59.69) (diameter 0) (color 0 0 0 0)
+  )
+  (junction (at 125.73 64.77) (diameter 0) (color 0 0 0 0)
+  )
+  (junction (at 142.24 59.69) (diameter 0) (color 0 0 0 0)
+  )
+  (junction (at 76.2 52.07) (diameter 0) (color 0 0 0 0)
+  )
+  (wire (pts (xy 157.48 59.69) (xy 157.48 60.96))
+    (stroke (width 0) (type default) (color 0 0 0 0))
+  )
+  (wire (pts (xy 121.92 57.15) (xy 124.46 57.15))
+    (stroke (width 0) (type default) (color 0 0 0 0))
+  )
+  (wire (pts (xy 106.68 64.77) (xy 125.73 64.77))
+    (stroke (width 0) (type default) (color 0 0 0 0))
+  )
+  (wire (pts (xy 76.2 52.07) (xy 76.2 53.34))
+    (stroke (width 0) (type default) (color 0 0 0 0))
+  )
+  (wire (pts (xy 88.9 52.07) (xy 91.44 52.07))
+    (stroke (width 0) (type default) (color 0 0 0 0))
+  )
+  (wire (pts (xy 130.81 67.31) (xy 130.81 64.77))
+    (stroke (width 0) (type default) (color 0 0 0 0))
+  )
+  (wire (pts (xy 142.24 54.61) (xy 142.24 59.69))
+    (stroke (width 0) (type default) (color 0 0 0 0))
+  )
+  (wire (pts (xy 88.9 59.69) (xy 91.44 59.69))
+    (stroke (width 0) (type default) (color 0 0 0 0))
+  )
+  (wire (pts (xy 76.2 48.26) (xy 76.2 52.07))
+    (stroke (width 0) (type default) (color 0 0 0 0))
+  )
+  (wire (pts (xy 139.7 59.69) (xy 142.24 59.69))
+    (stroke (width 0) (type default) (color 0 0 0 0))
+  )
+  (wire (pts (xy 130.81 64.77) (xy 125.73 64.77))
+    (stroke (width 0) (type default) (color 0 0 0 0))
+  )
+  (wire (pts (xy 121.92 52.07) (xy 157.48 52.07))
+    (stroke (width 0) (type default) (color 0 0 0 0))
+  )
+  (wire (pts (xy 88.9 52.07) (xy 88.9 57.15))
+    (stroke (width 0) (type default) (color 0 0 0 0))
+  )
+  (wire (pts (xy 142.24 59.69) (xy 144.78 59.69))
+    (stroke (width 0) (type default) (color 0 0 0 0))
+  )
+  (wire (pts (xy 137.16 59.69) (xy 139.7 59.69))
+    (stroke (width 0) (type default) (color 0 0 0 0))
+  )
+  (wire (pts (xy 91.44 57.15) (xy 88.9 57.15))
+    (stroke (width 0) (type default) (color 0 0 0 0))
+  )
+  (wire (pts (xy 121.92 54.61) (xy 142.24 54.61))
+    (stroke (width 0) (type default) (color 0 0 0 0))
+  )
+  (wire (pts (xy 139.7 67.31) (xy 130.81 67.31))
+    (stroke (width 0) (type default) (color 0 0 0 0))
+  )
+  (wire (pts (xy 121.92 59.69) (xy 124.46 59.69))
+    (stroke (width 0) (type default) (color 0 0 0 0))
+  )
+  (wire (pts (xy 76.2 52.07) (xy 88.9 52.07))
+    (stroke (width 0) (type default) (color 0 0 0 0))
+  )
+  (hierarchical_label "Mode 3V3" (shape input) (at 88.9 59.69 180)
+    (effects (font (size 1.27 1.27)) (justify right))
+  )
+  (hierarchical_label "V bat" (shape input) (at 76.2 48.26 0)
+    (effects (font (size 1.27 1.27)) (justify left))
+  )
+  (hierarchical_label "3V3_REG_RESET" (shape input) (at 124.46 57.15 0)
+    (effects (font (size 1.27 1.27)) (justify left))
+  )
+  (hierarchical_label "Vout 3.3V" (shape input) (at 144.78 59.69 0)
+    (effects (font (size 1.27 1.27)) (justify left))
+  )
+  (symbol (lib_id "Device:C") (at 139.7 63.5 0) (unit 1)
+    (in_bom yes) (on_board yes)
+    (property "Reference" "Cout" (id 0) (at 140.97 60.96 0)
+      (effects (font (size 1.27 1.27)) (justify left))
+    )
+    (property "Value" "22uF" (id 1) (at 140.97 66.04 0)
+      (effects (font (size 1.27 1.27)) (justify left))
+    )
+    (property "Footprint" "" (id 2) (at 140.6652 67.31 0)
+      (effects (font (size 1.27 1.27)) hide)
+    )
+    (property "Datasheet" "~" (id 3) (at 139.7 63.5 0)
+      (effects (font (size 1.27 1.27)) hide)
+    )
+    (pin "1")
+    (pin "2")
+  )
+  (symbol (lib_id "Device:C") (at 157.48 55.88 0) (unit 1)
+    (in_bom yes) (on_board yes) (fields_autoplaced)
+    (property "Reference" "Cvcc" (id 0) (at 161.29 54.6099 0)
+      (effects (font (size 1.27 1.27)) (justify left))
+    )
+    (property "Value" "1uF " (id 1) (at 161.29 57.1499 0)
+      (effects (font (size 1.27 1.27)) (justify left))
+    )
+    (property "Footprint" "" (id 2) (at 158.4452 59.69 0)
+      (effects (font (size 1.27 1.27)) hide)
+    )
+    (property "Datasheet" "~" (id 3) (at 157.48 55.88 0)
+      (effects (font (size 1.27 1.27)) hide)
+    )
+    (pin "1")
+    (pin "2")
+  )
+  (symbol (lib_id "pspice:INDUCTOR") (at 130.81 59.69 0) (unit 1)
+    (in_bom yes) (on_board yes)
+    (property "Reference" "L1" (id 0) (at 124.46 62.23 0))
+    (property "Value" "68uH" (id 1) (at 130.81 62.23 0))
+    (property "Footprint" "" (id 2) (at 130.81 59.69 0)
+      (effects (font (size 1.27 1.27)) hide)
+    )
+    (property "Datasheet" "~" (id 3) (at 130.81 59.69 0)
+      (effects (font (size 1.27 1.27)) hide)
+    )
+    (pin "1")
+    (pin "2")
+  )
+  (symbol (lib_id "power:GND") (at 157.48 60.96 0) (unit 1)
+    (in_bom yes) (on_board yes) (fields_autoplaced)
+    (property "Reference" "#PWR?" (id 0) (at 157.48 67.31 0)
+      (effects (font (size 1.27 1.27)) hide)
+    )
+    (property "Value" "GND" (id 1) (at 157.48 66.04 0))
+    (property "Footprint" "" (id 2) (at 157.48 60.96 0)
+      (effects (font (size 1.27 1.27)) hide)
+    )
+    (property "Datasheet" "" (id 3) (at 157.48 60.96 0)
+      (effects (font (size 1.27 1.27)) hide)
+    )
+    (pin "1")
+  )
+  (symbol (lib_id "Device:C") (at 76.2 57.15 0) (unit 1)
+    (in_bom yes) (on_board yes)
+    (property "Reference" "Cin" (id 0) (at 71.12 55.88 0)
+      (effects (font (size 1.27 1.27)) (justify left))
+    )
+    (property "Value" "1 uF" (id 1) (at 69.85 59.69 0)
+      (effects (font (size 1.27 1.27)) (justify left))
+    )
+    (property "Footprint" "" (id 2) (at 77.1652 60.96 0)
+      (effects (font (size 1.27 1.27)) hide)
+    )
+    (property "Datasheet" "~" (id 3) (at 76.2 57.15 0)
+      (effects (font (size 1.27 1.27)) hide)
+    )
+    (pin "1")
+    (pin "2")
+  )
+  (symbol (lib_id "Regulator_Switching_MAX17640AATA:MAX17640AATA") (at 106.68 54.61 0) (unit 1)
+    (in_bom yes) (on_board yes) (fields_autoplaced)
+    (property "Reference" "U?" (id 0) (at 111.76 44.45 0))
+    (property "Value" "MAX17640AATA" (id 1) (at 111.76 46.99 0))
+    (property "Footprint" "" (id 2) (at 106.68 54.61 0)
+      (effects (font (size 1.27 1.27)) hide)
+    )
+    (property "Datasheet" "https://www.mouser.com/datasheet/2/256/MAX17640-2399981.pdf" (id 3) (at 106.68 54.61 0)
+      (effects (font (size 1.27 1.27)) hide)
+    )
+    (pin "1")
+    (pin "2")
+    (pin "3")
+    (pin "4")
+    (pin "5")
+    (pin "6")
+    (pin "7")
+    (pin "8")
+  )
+  (symbol (lib_id "power:GND") (at 76.2 60.96 0) (unit 1)
+    (in_bom yes) (on_board yes)
+    (property "Reference" "#PWR?" (id 0) (at 76.2 67.31 0)
+      (effects (font (size 1.27 1.27)) hide)
+    )
+    (property "Value" "GND" (id 1) (at 76.2 64.77 0))
+    (property "Footprint" "" (id 2) (at 76.2 60.96 0)
+      (effects (font (size 1.27 1.27)) hide)
+    )
+    (property "Datasheet" "" (id 3) (at 76.2 60.96 0)
+      (effects (font (size 1.27 1.27)) hide)
+    )
+    (pin "1")
+  )
+  (symbol (lib_id "power:GND") (at 125.73 64.77 0) (unit 1)
+    (in_bom yes) (on_board yes) (fields_autoplaced)
+    (property "Reference" "#PWR?" (id 0) (at 125.73 71.12 0)
+      (effects (font (size 1.27 1.27)) hide)
+    )
+    (property "Value" "GND" (id 1) (at 125.73 69.85 0))
+    (property "Footprint" "" (id 2) (at 125.73 64.77 0)
+      (effects (font (size 1.27 1.27)) hide)
+    )
+    (property "Datasheet" "" (id 3) (at 125.73 64.77 0)
+      (effects (font (size 1.27 1.27)) hide)
+    )
+    (pin "1")
+  )
 )

Commit message: finished template stuff
Parts:
- gave numbers to parts that had none: 1
- renumbered Cin to Cin701, Cout to Cout701, Cvcc to Cvcc701, L1 to L701
Changed lines of the file:
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@@
   (symbol (lib_id "Device:C") (at 139.7 63.5 0) (unit 1)
     (in_bom yes) (on_board yes)
-    (property "Reference" "Cout" (id 0) (at 140.97 60.96 0)
+    (property "Reference" "Cout701" (id 0) (at 140.97 60.96 0)
       (effects (font (size 1.27 1.27)) (justify left))
     )
@@
   (symbol (lib_id "Device:C") (at 157.48 55.88 0) (unit 1)
     (in_bom yes) (on_board yes) (fields_autoplaced)
-    (property "Reference" "Cvcc" (id 0) (at 161.29 54.6099 0)
+    (property "Reference" "Cvcc701" (id 0) (at 161.29 54.6099 0)
       (effects (font (size 1.27 1.27)) (justify left))
     )
@@
   (symbol (lib_id "pspice:INDUCTOR") (at 130.81 59.69 0) (unit 1)
     (in_bom yes) (on_board yes)
-    (property "Reference" "L1" (id 0) (at 124.46 62.23 0))
+    (property "Reference" "L701" (id 0) (at 124.46 62.23 0))
     (property "Value" "68uH" (id 1) (at 130.81 62.23 0))
     (property "Footprint" "" (id 2) (at 130.81 59.69 0)
@@
   (symbol (lib_id "power:GND") (at 157.48 60.96 0) (unit 1)
     (in_bom yes) (on_board yes) (fields_autoplaced)
-    (property "Reference" "#PWR?" (id 0) (at 157.48 67.31 0)
+    (property "Reference" "#PWR0702" (id 0) (at 157.48 67.31 0)
       (effects (font (size 1.27 1.27)) hide)
     )
@@
   (symbol (lib_id "Device:C") (at 76.2 57.15 0) (unit 1)
     (in_bom yes) (on_board yes)
-    (property "Reference" "Cin" (id 0) (at 71.12 55.88 0)
+    (property "Reference" "Cin701" (id 0) (at 71.12 55.88 0)
       (effects (font (size 1.27 1.27)) (justify left))
     )
@@
   (symbol (lib_id "Regulator_Switching_MAX17640AATA:MAX17640AATA") (at 106.68 54.61 0) (unit 1)
     (in_bom yes) (on_board yes) (fields_autoplaced)
-    (property "Reference" "U?" (id 0) (at 111.76 44.45 0))
+    (property "Reference" "U701" (id 0) (at 111.76 44.45 0))
     (property "Value" "MAX17640AATA" (id 1) (at 111.76 46.99 0))
     (property "Footprint" "" (id 2) (at 106.68 54.61 0)
@@
   (symbol (lib_id "power:GND") (at 76.2 60.96 0) (unit 1)
     (in_bom yes) (on_board yes)
-    (property "Reference" "#PWR?" (id 0) (at 76.2 67.31 0)
+    (property "Reference" "#PWR0701" (id 0) (at 76.2 67.31 0)
       (effects (font (size 1.27 1.27)) hide)
     )
@@
   (symbol (lib_id "power:GND") (at 125.73 64.77 0) (unit 1)
     (in_bom yes) (on_board yes) (fields_autoplaced)
-    (property "Reference" "#PWR?" (id 0) (at 125.73 71.12 0)
+    (property "Reference" "#PWR0703" (id 0) (at 125.73 71.12 0)
       (effects (font (size 1.27 1.27)) hide)
     )
