File: boards/TARS-MK4/TARS-MK4-FCB-revB/TARS-MK4-FCB.kicad_pcb (KiCad board)
At the start: 2 copper layers, 86 x 79.1 mm, 70 parts, among them J101 U.FL, J102 Molex_SlimStack_2091680401_2x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, J103 Molex_SlimStack_2091680401_2x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, J104 Molex_SlimStack_Plug_2x20_P0.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, J105 Molex_SlimStack_Plug_2x20_P0.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, J106 Conn_01x03, J107 Conn_01x02, J108 Conn_01x06, J109 Conn_01x03, Q101 SSM3K16FU, SW101 FSMSM Switch, U101 MS5611-01BA03, U102 LSM6DSLTR, U103 MAX-M10S, U104 BNO086, U105 LIS3MDL, U106 KX134-1211, U107 Teensy4.1, U108 BME688, Y101 32.768kHz

Commit message: Updated Silkscreens
Other:
- board text added: "Flight Computation Board Rev.B"
- board text removed: "Flight Computation Board Rev.A"
Changed lines of the file:
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@@
     (effects (font (size 0.5 0.5) (thickness 0.12)) (justify mirror))
   )
-  (gr_text "Flight Computation Board Rev.A" (at 114.15 81.22) (layer "B.SilkS")
+  (gr_text "Flight Computation Board Rev.B" (at 114.15 81.22) (layer "B.SilkS")
     (effects (font (size 1 1) (thickness 0.2)) (justify mirror))
   )

Commit message: Fixed solder mask, now 0mm
Other:
- rule pad_to_mask_clearance: 0.254 -> 0
Changed lines of the file:
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@@
       (dielectric_constraints no)
     )
-    (pad_to_mask_clearance 0.254)
+    (pad_to_mask_clearance 0)
     (pcbplotparams
       (layerselection 0x00010fc_ffffffff)
