File: boards/TRACKER/TRACKER-MK1/TRACKER-MK1.kicad_pcb (KiCad board)
At the start: 2 copper layers, 60 x 90 mm, 126 parts, among them J101 1054500101, J102 1040310811, J103 JST-PH, J104 JST-PH, J105 JST-PH, J106 JST-PH, J107 JST-PH, J108 JST-PH, J109 JST-PH, J110 2.54mm Pin Header, J111 2.54mm Pin Header, J112 JST-PH, J113 JST-PH, J114 JST-PH, J115 JST-PH, J116 U.FL, J117 2.54mm Pin Header, J120 2.54mm Pin Header, J121 2.54mm Pin Header, J122 2.54mm Pin Header, J123 2.54mm Pin Header, J124 2.54mm Pin Header, J125 2.54mm Pin Header, J126 2.54mm Pin Header, SW101 VBUS Switch, SW102 Battery Switch, SW103 Power Switch, SW104 SW_Push, SW105 SW_Push, U101 TCAL9539-Q1, U102 BQ25180, U103 ECMF02-2AMX6, U104 ADS7138-Q1, U105 ADP5589, U106 TPS566242DRLR, U107 ESP32-S3-WROOM-1, U108 BNO085, U109 SAM-M10Q-00B, U201 CC1125, X201 ECS-TXO-2016MV-400-TR

Commit message: Finalized MK1
Parts:
- removed J110: 2.54mm Pin Header, Connector_PinHeader_2.54mm:PinHeader_1x01_P2.54mm_Vertical
- removed J122: 2.54mm Pin Header, Connector_PinHeader_2.54mm:PinHeader_1x02_P2.54mm_Vertical
- removed J124: 2.54mm Pin Header, Connector_PinHeader_2.54mm:PinHeader_1x03_P2.54mm_Vertical
- C109, C110, C111, C113, R103: moved to F.Cu
- R107, R120, R121: moved to B.Cu
- moved J121 196.9 mm to (77.9, 39.8), turned to 180 degrees
- moved J123 184.5 mm to (77.5, 93.8), turned to -90 degrees
- moved J120 150.3 mm to (107.1, 91.7), turned to 90 degrees
- moved J125 131.1 mm to (119.0, 86.0), turned to 180 degrees
- moved C204 117.1 mm to (121.2, 49.7), turned to -90 degrees
- moved J116 116.9 mm to (124.9, 41.8), turned to 180 degrees
- moved C206 116.1 mm to (122.9, 49.7), turned to -90 degrees
- moved R202 112.8 mm to (121.2, 46.2), turned to -90 degrees
- moved C225 112.5 mm to (123.3, 37.5), turned to -90 degrees
- moved L206 112.3 mm to (118.8, 36.6)
- moved C221 112.1 mm to (121.5, 35.9)
- moved C205 111.7 mm to (122.9, 46.2), turned to -90 degrees
- moved C213 111.6 mm to (121.2, 41.5)
- moved C207 111.6 mm to (118.9, 43.8)
- moved L203 111.6 mm to (119.6, 41.5)
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Connections:
- J114 pad 1: /I2C_SNS_SDA -> /I2C_SNS_SCL
- J114 pad 2: /I2C_SNS_SCL -> /I2C_SNS_SDA
- J115 pad 1: /I2C_AUX_SDA -> /I2C_AUX_SCL
- J115 pad 2: /I2C_AUX_SCL -> /I2C_AUX_SDA
- J123 pad 1: /I2C_AUX_SDA -> /I2C_AUX_SCL
- J123 pad 2: /I2C_AUX_SCL -> /I2C_AUX_SDA
- U105 pad 1: Net-(J110-Pin_1) -> /TCAL_RESET
- U105 pad 2: /BQ25180_INT -> /TCAL_INT
- U105 pad 4: /TCAL_RESET -> /BQ25180_INT
Routing:
- net /3V3: track 125.4 -> 400.7 mm, vias 4 -> 19
- net /I2C_AUX_SDA: track 0.00 -> 191.0 mm, vias 0 -> 4
- net /I2C_AUX_SCL: track 0.00 -> 187.6 mm, vias 0 -> 5
- net /CC1125_GPIO0: track 0.00 -> 127.3 mm, vias 0 -> 4
- net /I2C_SNS_SCL: track 0.00 -> 124.2 mm, vias 0 -> 4
- net /I2C_SNS_SDA: track 0.00 -> 112.8 mm, vias 0 -> 4
- net /INT_GNSS: track 0.00 -> 111.8 mm, vias 0 -> 2
- net /SPI2_CC1125_~{CS}: track 0.00 -> 109.4 mm, vias 0 -> 3
- net /CC1125_GPIO3: track 0.00 -> 106.7 mm, vias 0 -> 3
- net /SPI2_RADIO_MOSI: track 0.00 -> 106.4 mm, vias 0 -> 3
- net /SPI2_RADIO_MISO: track 0.00 -> 105.4 mm, vias 0 -> 3
- net /CC1125_GPIO2: track 0.00 -> 103.0 mm, vias 0 -> 3
- net /SPI2_RADIO_CLK: track 0.00 -> 100.1 mm, vias 0 -> 3
- net /CC1125_~{RESET}: track 0.00 -> 88.0 mm, vias 0 -> 3
- net /ADP_~{INT}: track 0.00 -> 78.7 mm, vias 0 -> 3
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- removed copper zone on F.Cu, net /3V3
Other:
- board text added: "+"
- board text added: "-"
- board text added: "3V3"
- board text added: "ADP"
- board text added: "ADS GPIO"
- board text added: "Aux I2C"
- board text added: "B"
- board text added: "BNO085"
- board text added: "BOOT"
- board text added: "Battery"
- board text added: "Buzzer"
- board text added: "C1"
- board text added: "C10"
- board text added: "C2"
- board text added: "C3"
- board text added: "C4"
- board text added: "C5"
- board text added: "C6"
- board text added: "C7"
- board text added: "C8"
- board text added: "C9"
- board text added: "CC1125 Radio"
- board text added: "CLK"
- board text added: "CMD"
- board text added: "CS"
- board text added: "DAT0"
- board text added: "DAT1"
- board text added: "DAT2"
- board text added: "DAT3"
- board text added: "DCS"
- board text added: "DISP"
- board text added: "DMOSI"
- board text added: "DSCLK"
- board text added: "D_3V3"
- board text added: "Display"
- board text added: "ESP32"
- board text added: "EXINT"
- board text added: "EXTMD"
- board text added: "GND"
- board text added: "GPI00"
- board text added: "GPI02"
- board text added: "GPI03"
- board text added: "GPIO0"
- board text added: "GPIO1"
- board text added: "GPIO2"
- board text added: "GPIO3"
- board text added: "GPIO4"
- board text added: "GPIO5"
- board text added: "GPIO6"
- board text added: "GPIO7"
- board text added: "GPS"
- board text added: "INT"
- board text added: "INT_GNSS"
- board text added: "Keypad"
- board text added: "MISO"
- board text added: "MOSI"
- board text added: "NC"
- board text added: "NOT POWER INPUT"
- board text added: "P01"
- board text added: "P02"
- board text added: "P03"
- board text added: "P04"
- board text added: "P05"
- board text added: "P06"
- board text added: "P07"
- board text added: "P10"
- board text added: "P11"
- board text added: "P12"
- board text added: "P13"
- board text added: "P14"
- board text added: "P15"
- board text added: "P16"
- board text added: "P17"
- board text added: "PWM"
- board text added: "Peter Giannetos"
- board text added: "R"
- board text added: "R1"
- board text added: "R2"
- board text added: "R3"
- board text added: "R4"
- board text added: "RESET"
- board text added: "RevA"
- board text added: "SCL"
- board text added: "SD CARD"
- board text added: "SDA"
- board text added: "SNS I2C"
- board text added: "Switch Battery"
- board text added: "Switch Power"
- board text added: "Switch USB Power"
- board text added: "TCAL GPIO"
- board text added: "TIME"
- board text added: "TRACKER MK1"
- board text added: "TS/MR"
- board text added: "Thermistor"
- board text added: "VBAT+"
- board text added: "VBUS"
- board text added: "VBUS+"
- board text added: "VSYS"
- board text added: "VSYS+"
- board text added: "WayWayWay"
