File: boards/SPARK-MK1/SPARK-MK1.kicad_sch (KiCad schematic)
At the start: 72 parts, among them J1 Screw_Terminal_01x02, J101 Conn_01x03_Pin, J102 Screw_Terminal_01x02, J103 Screw_Terminal_01x02, J104 Conn_01x03_Pin, J105 Conn_01x03_Pin, J106 Screw_Terminal_01x02, J107 Screw_Terminal_01x02, J109 Conn_01x04_Pin, J110 Conn_01x02_Pin, J111 Conn_01x04_Pin, J112 Conn_01x04_Pin, J113 Conn_01x03_Pin, J2 Screw_Terminal_01x02, J3 Screw_Terminal_01x02, J4 Screw_Terminal_01x02, U1 AD5252BRUZ1, U101 AD5252BRUZ1, U2 Teensy4.1_bare, U5 TPS25947, U6 TPS25947, U7 TPS25947, U8 TPS25947

Commit message: Commiting
Parts:
- removed J101, J104, J105, J113: Conn_01x03_Pin, Connector_PinHeader_2.54mm:PinHeader_1x03_P2.54mm_Vertical, symbol Connector:Conn_01x03_Pin
- removed J109, J111, J112: Conn_01x04_Pin, Connector_PinHeader_2.54mm:PinHeader_1x04_P2.54mm_Vertical, symbol Connector:Conn_01x04_Pin
- removed J110: Conn_01x02_Pin, Connector_PinHeader_2.54mm:PinHeader_1x02_P2.54mm_Vertical, symbol Connector:Conn_01x02_Pin
- added J101, J104, J105, J112: Conn_01x03, Connector_PinHeader_2.54mm:PinHeader_1x03_P2.54mm_Vertical, symbol Connector_Generic:Conn_01x03
- added J108: Conn_01x02, Connector_PinHeader_2.54mm:PinHeader_1x02_P2.54mm_Vertical, symbol Connector_Generic:Conn_01x02
- added J109, J110, J111: Conn_01x04, Connector_PinHeader_2.54mm:PinHeader_1x04_P2.54mm_Vertical, symbol Connector_Generic:Conn_01x04
Connections:
- net B1_A: now also J110.2 (Pin_2), J112.2 (Pin_2)
- net B1_B: now also J104.2 (Pin_2), J109.2 (Pin_2)
- net B3_A: now also J101.2 (Pin_2), J110.4 (Pin_4)
- net B3_B: now also J105.2 (Pin_2), J109.4 (Pin_4)
- net DiPot_A_A0: now also J111.3 (Pin_3)
- net DiPot_A_A1: now also J111.4 (Pin_4)
- net DiPot_B_A0: now also J111.1 (Pin_1)
- net DiPot_B_A1: now also J111.2 (Pin_2)
- net GND: now also J109.1 (Pin_1), J109.3 (Pin_3), J110.1 (Pin_1), J110.3 (Pin_3)
- net I2C_SCL: now also J108.2 (Pin_2)
- net I2C_SDA: now also J108.1 (Pin_1)
- net PG_EF_A: now also J112.3 (Pin_3)
- net PG_EF_B: now also J101.3 (Pin_3)
- net PG_EF_C: now also J104.3 (Pin_3)
- net PG_EF_D: now also J105.3 (Pin_3)
- net PYRO_A_OUT: now also J112.1 (Pin_1)
- net PYRO_B_OUT: now also J101.1 (Pin_1)
- net PYRO_C_OUT: now also J104.1 (Pin_1)
- net PYRO_D_OUT: now also J105.1 (Pin_1)

Commit message: schem and lib fixes
Parts:
- added C13, C3: 100 nF, Capacitor_SMD:C_0603_1608Metric, symbol Device:C
- added C14, C4: 1 uF, Capacitor_SMD:C_0603_1608Metric, symbol Device:C
- C101, C102, C103, C104, C11, C12, C7, C8: symbol Device:C_Polarized_US -> Device:C
- U1, U101: footprint AD5252BRUZ10-RL7:RU_14_ADI-M -> AD5252BRUZ1:SOP65P640X120-14N
- U2: footprint Teensy4.1bare:Teensy_4.1 -> Teensy4.1bare:Teensy41_bare_pins
Connections:
- net GND: now also C13.2, C14.2, C3.2, C4.2
- net 3V3 renamed +3V3
- net +3V3: now also C13.1, C14.1, C3.1, C4.1
- no-connect marks 37 -> 40
Other:
- note added: "Input Screw Terminals"
- note added: "Output Screw Terminals"
- note removed: "Screw Terminals"
- moved on the sheet: BZ101, C10, C6, C9, D101, D102, D103, D104, H101, H102, H103, H104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
