File: boards/Feather_Duo/Feather_Duo.kicad_sch (KiCad schematic)
At the start: 32 parts, among them J101 Conn_01x04, J102 Conn_01x04, J103 Conn_01x03, J104 Conn_01x04, J105 Conn_01x04, J106 USB4105-GF-A, J107 Conn_01x04, U101 ESP32-S3-MINI-1U, U102 ECMF02-2AMX6, U103 AMS1117-3.3

Commit message: library + metadata changes
Other:
- company: (none) -> Illinois Space Society
- title: (none) -> Feather Duo
Changed lines of the file:
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@@
 	(paper "A4")
 	(title_block
+		(title "Feather Duo")
+		(date "2/14/2025")
+		(rev "A")
+		(company "Illinois Space Society")
 		(comment 4 "Contributors: Nicholas Phillips, Thomas McManamen")
 	)
@@
 		)
 		(instances
-			(project "Feather1268"
+			(project "Feather_Duo"
 				(path "/69669038-9204-4ef2-bc4f-06a0bd7ceaf5"
 					(page "2")
@@
 		)
 		(instances
-			(project "Feather1268"
+			(project "Feather_Duo"
 				(path "/69669038-9204-4ef2-bc4f-06a0bd7ceaf5"
 					(page "3")
