File: boards/EAGLE-MK1/EAGLE-MK1-revA/EAGLE-MK1-revA.kicad_pcb (KiCad board)
At the start: 4 copper layers, 50 x 55 mm, 73 parts, among them J1 SMA, J101 USB4105-GF-A, J107 Conn_01x03, J108 Conn_01x03, J109 Conn_01x03, SW2 SW_Push, SW3 SW_Push, U1 RF4463PRO, U101 ECMF02-2AMX6, U106 INA745x, U2 TPS63802, U4 PMA-545G1+, U5 TPSM82813, U7 ESP32-P4

Commit message: ROUTING DONE
New LR2021 Footprint Integration
Parts:
- U1: value RF4463PRO -> LR2021; footprint RF_Module_NiceRF:RF4463PRO -> RF_Module_NiceRF:LR2021
- U2: footprint Package_DFN:DLA0010A -> Package_SON_ISS:VSON-HR-DLA0010A
- U7: footprint MCU_ESP32:ESP32-P4-Module-Waveshare -> MCU_ESP32:ESP32-P4-Module
- moved C31 22.7 mm to (129.4, 123.9), turned to 180 degrees
- moved U7 18.7 mm to (143.3, 91.9)
- moved C10 17.5 mm to (133.6, 123.9), turned to 0 degrees
- moved C35 7.60 mm to (151.9, 117.6)
- moved C33 3.39 mm to (154.6, 119.9)
- moved C34 3.32 mm to (152.2, 120.7)
- moved R4 3.29 mm to (152.2, 119.2)
- moved C36 3.16 mm to (157.6, 111.8)
- moved C37 3.16 mm to (152.7, 114.8)
- moved L1 3.16 mm to (155.6, 111.5)
- moved L2 3.16 mm to (153.4, 111.5)
- moved U4 3.16 mm to (156.0, 115.9)
- moved R119 2.44 mm to (156.3, 120.0), turned to 90 degrees
- moved R118 2.43 mm to (159.3, 116.1)
- moved C49 2.40 mm to (160.8, 116.1)
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Connections:
- net /Antenna_Connector_T renamed /Amplifer_Input
- C37 pad 1: /Si4463_ANT -> /LR2021_ANT
- R119 pad 1: /Si4463_ANT -> /LR2021_ANT
- U1 pad 1: GND -> +3V3
- U1 pad 10: /Si4463_nIRQ -> unconnected-(U1-2.4_ANT-Pad10)
- U1 pad 11: /Si4463_EN -> GND
- U1 pad 13: GND -> unconnected-(U1-VTCXO-Pad13)
- U1 pad 14: /Si4463_ANT -> /LR2021_nRST
- U1 pad 2: unconnected-(U1-NC-Pad2) -> GND
- U1 pad 3: /Si4463_GPIO0 -> /SPI_MISO
- U1 pad 4: /Si4463_GPIO1 -> /SPI_MOSI
- U1 pad 5: +3V3 -> /SPI_SCK
- U1 pad 6: /SPI_MISO -> /LR2021_CS
- U1 pad 7: /SPI_MOSI -> /LR2021_BUSY
- U1 pad 8: /SPI_SCK -> GND
- U1 pad 9: /Si4463_CS -> /LR2021_ANT
- U7 pad 19: unconnected-(U7-GPIO4-Pad19) -> /LR2021_DIO9
- U7 pad 20: /Si4463_EN -> /LR2021_BUSY
- U7 pad 21: /Si4463_nIRQ -> /LR2021_nRST
- U7 pad 22: /Si4463_CS -> /LR2021_CS
- U7 pad 26: /Si4463_GPIO1 -> /LR2021_DIO7
- U7 pad 27: /Si4463_GPIO0 -> /LR2021_DIO8
Routing:
- net /LR2021_BUSY: track 0.00 -> 28.0 mm
- net /LR2021_CS: track 0.00 -> 24.4 mm
- net /SPI_SCK: track 14.5 -> 36.7 mm, vias 0 -> 2
- net /Si4463_ANT: track 20.1 -> 0.00 mm
- net /LR2021_ANT: track 0.00 -> 18.9 mm
- net /LR2021_nRST: track 0.00 -> 15.2 mm, vias 0 -> 2
- net /SPI_MOSI: track 17.3 -> 31.3 mm, vias 0 -> 2
- net /LR2021_DIO9: track 0.00 -> 13.1 mm, vias 0 -> 2
- net /Si4463_GPIO1: track 8.81 -> 0.00 mm, vias 2 -> 0
- net /Si4463_GPIO0: track 8.76 -> 0.00 mm, vias 2 -> 0
- net /Si4463_EN: track 8.54 -> 0.00 mm
- net /Si4463_nIRQ: track 7.97 -> 0.00 mm
- net /Si4463_CS: track 7.36 -> 0.00 mm
- net GND: track 3.84 -> 9.31 mm, vias 218 -> 212
- net /LR2021_DIO7: track 0.00 -> 3.73 mm
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Other:
- board text added: "REVB"

Commit message: a
Routing:
- net GND: vias 212 -> 216
Changed lines of the file:
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@@
 	)
 	(via
+		(at 131.4 105.29)
+		(size 0.6)
+		(drill 0.3)
+		(layers "F.Cu" "B.Cu")
+		(free yes)
+		(net 2)
+	)
+	(via
 		(at 166.75 109.425)
 		(size 0.6)
@@
 	)
 	(via
+		(at 132.95 108.89)
+		(size 0.6)
+		(drill 0.3)
+		(layers "F.Cu" "B.Cu")
+		(free yes)
+		(net 2)
+	)
+	(via
 		(at 129.475 87.625)
 		(size 0.6)
@@
 	)
 	(via
+		(at 132.56 100.58)
+		(size 0.6)
+		(drill 0.3)
+		(layers "F.Cu" "B.Cu")
+		(free yes)
+		(net 2)
+	)
+	(via
 		(at 148.85 110.65)
 		(size 0.6)
@@
 	)
 	(via
+		(at 133.36 102.53)
+		(size 0.6)
+		(drill 0.3)
+		(layers "F.Cu" "B.Cu")
+		(free yes)
+		(net 2)
+	)
+	(via
 		(at 150.25 105.85)
 		(size 0.6)
@@
 	(segment
 		(start 135.798159 101.4)
+		(end 132.8 101.4)
+		(width 0.2)
+		(layer "B.Cu")
+		(net 139)
+	)
+	(segment
+		(start 132.8 101.4)
 		(end 129.55 101.4)
 		(width 0.2)
